Commit message: holy crap it drove through it

File: src/project/project_description/urdf/project.gazebo.xacro (robot description, xacro)
@@ -20,5 +20,5 @@
     </gazebo>
     <!-- Camera Plugin -->
-    <xacro:property name="camera_update_hz" value="10" />
+    <xacro:property name="camera_update_hz" value="60" />
     <gazebo reference="camera">
         <sensor type="camera" name="camera1">
